Commit message: Increased mass for base component and used black for the printed parts

File: SCARA.urdf (robot description, URDF)
Before this commit: robot URDF, 25 links, 24 joints
Links:
- removed link z_stepper
- added link l1_stepper, mass 0.5336531870485284; collision mesh filename=CAD/stepper.stl scale=0.001 0.001 0.001; visual mesh filename=CAD/stepper.stl scale=0.001 0.001 0.001
- link base: mass 4.290391579347167 -> 100
Joints:
- removed joint z_stepper_Rigido-13
- added joint l1_stepper_Rigido-13: type fixed, parent l1_stepper, child coupler, origin xyz=-0.015494 -0.015494 -0.024000000000000004 rpy=-3.141592653589793 -0.0 1.298208104246751e-67
- joint z_axis_mount_Rigido-4: child z_stepper -> l1_stepper

Commit message: Updated urdf

File: SCARA.urdf (robot description, URDF)
Before this commit: robot URDF, 25 links, 24 joints
Joints:
- removed joint anti_wobble_Rigido-22
- removed joint base_Rigido-3
- removed joint coupler_Rigido-5
- removed joint ee_51105_bearing_Rivoluzione-28
- removed joint l1_platform_bottom_Rigido-11
- removed joint l1_platform_bottom_Rigido-14
- removed joint l1_platform_bottom_Rigido-17
- removed joint l1_platform_bottom_Rigido-21
- removed joint l1_stepper_Rigido-13
- removed joint l2_51105_bearing_Rivoluzione-19
- removed joint l2_bottom_Rigido-24
- removed joint l2_top_Rigido-20
- removed joint l2_top_Rigido-23
- removed joint l3_51105_bearing_Rivoluzione-25
- removed joint l3_bottom_Rigido-27
- removed joint l3_bottom_Rigido-29
- removed joint l3_top_Rigido-26
- removed joint linear_rod_4_Rigido-15
- removed joint z_axis_mount_Rigido-10
- removed joint z_axis_mount_Rigido-4
- removed joint z_axis_mount_Rigido-7
- removed joint z_axis_mount_Rigido-8
- removed joint z_axis_mount_Rigido-9
- removed joint z_axis_mount_Scorrimento-31
- added joint anti_wobble_608_bearing: type fixed, parent anti_wobble, child 608_bearing, origin xyz=-0.03 -0.021499999999999995 0.01 rpy=3.141592653589793 8.930854384075464e-79 9.056962336419341e-48
- added joint base_z_axis_mount: type fixed, parent base, child z_axis_mount, origin xyz=0.026000000000000002 -0.0275 0.111 rpy=3.141592653589793 -0.0 0.0
- added joint coupler_leadscrew: type fixed, parent coupler, child leadscrew, origin xyz=0.0 0.0 0.015399999999999992 rpy=-1.232595164407831e-32 2.465190328815662e-32 2.1271369958606197e-63
- added joint ee_51105_bearing_ee_mount: type revolute, parent ee_51105_bearing, child ee_mount, origin xyz=-1.084365242088408e-33 0.0 0.010996769999999998 rpy=2.465190328815662e-32 -6.162975822039155e-33 -1.2228926112448176e-33, axis 6.162975822039155e-33 2.465190328815662e-32 1.0, limit lower=0.0 upper=5.585054 effort=1000 velocity=1000000
- added joint l1_platform_bottom_l1_T8_nut: type fixed, parent l1_platform_bottom, child l1_T8_nut, origin xyz=-0.038 0.021499999999999995 0.006000000000000014 rpy=-3.141592653589793 -0.0 -3.575378658000282e-49
- added joint l1_platform_bottom_l1_platform_top: type fixed, parent l1_platform_bottom, child l1_platform_top, origin xyz=-0.061 0.020999999999999998 0.02400000000000002 rpy=6.162975822039155e-33 -0.0 -3.575378658000282e-49
- added joint l1_platform_bottom_l2_51105_bearing: type fixed, parent l1_platform_bottom, child l2_51105_bearing, origin xyz=-0.03 -0.03900000000000001 0.0010000000000000143 rpy=-3.141592653589793 -0.0 -3.575378658000282e-49
- added joint l1_platform_bottom_l2_stepper: type fixed, parent l1_platform_bottom, child l2_stepper, origin xyz=-0.0455 0.0405 0.0 rpy=-3.141592653589793 -0.0 -3.575378658000282e-49
- added joint l1_stepper_coupler: type fixed, parent l1_stepper, child coupler, origin xyz=-0.015494 -0.015494 -0.024000000000000004 rpy=-3.141592653589793 -0.0 1.298208104246751e-67
- added joint l2_51105_bearing_l2_top: type revolute, parent l2_51105_bearing, child l2_top, origin xyz=-2.710913105221029e-34 0.0 0.010996770000000015 rpy=-6.162975822039155e-33 -2.6317740138327936e-81 -4.2702974826242526e-49, axis -0.0 0.0 1.0, limit lower=0.0 upper=3.141593 effort=1000 velocity=1000000
- added joint l2_bottom_l3_51105_bearing: type fixed, parent l2_bottom, child l3_51105_bearing, origin xyz=0.03 -0.024000000000000004 -0.030999999999999996 rpy=0.0 -2.4781487288111424e-80 4.0210262061213034e-48
- added joint l2_top_l2_bottom: type fixed, parent l2_top, child l2_bottom, origin xyz=0.09 -0.024000000000000004 0.005999999999999997 rpy=3.141592653589793 -0.0 -5.503376651748532e-48
- added joint l2_top_l3_stepper: type fixed, parent l2_top, child l3_stepper, origin xyz=0.0325 -0.015499999999999998 0.0 rpy=3.141592653589793 -0.0 -5.503376651748532e-48
- added joint l3_51105_bearing_l3_top: type revolute, parent l3_51105_bearing, child l3_top, origin xyz=0.0 0.0 -0.010996760000000006 rpy=6.162975822039155e-33 -6.162975822039155e-33 -1.2228926112447996e-33, axis -6.162975822039155e-33 -0.0 -1.0, limit lower=-1.22173 upper=4.712389 effort=1000 velocity=1000000
- added joint l3_bottom_ee_51105_bearing: type fixed, parent l3_bottom, child ee_51105_bearing, origin xyz=-0.03 0.024000000000000004 -0.030999999999999996 rpy=3.141592653589793 -0.0 -6.310936878636713e-46
- added joint l3_bottom_ee_stepper: type fixed, parent l3_bottom, child ee_stepper, origin xyz=0.016500000000000004 0.008499999999999997 -0.031999999999999994 rpy=3.141592653589793 -0.0 -6.310936878636713e-46
- added joint l3_top_l3_bottom: type fixed, parent l3_top, child l3_bottom, origin xyz=-0.09 -0.024000000000000004 -0.005999999999999997 rpy=-6.117533459552187e-64 6.162975822039155e-33 1.2228926112447658e-33
- added joint linear_rod_4_anti_wobble: type fixed, parent linear_rod_4, child anti_wobble, origin xyz=0.0 0.0 -0.3 rpy=9.860761315262648e-32 -0.0 0.0
- added joint z_axis_mount_l1_platform_bottom: type prismatic, parent z_axis_mount, child l1_platform_bottom, origin xyz=0.003999999999999999 0.013499999999999996 -0.046 rpy=3.141592653589793 -0.0 0.0, axis 0.0 0.0 1.0, limit lower=0.0 upper=0.18 effort=1000 velocity=1000000
- added joint z_axis_mount_l1_stepper: type fixed, parent z_axis_mount, child l1_stepper, origin xyz=-0.0105 0.0075 0.0 rpy=0.0 -0.0 0.0
- added joint z_axis_mount_linear_rod_1: type fixed, parent z_axis_mount, child linear_rod_1, origin xyz=-0.055999999999999994 0.013499999999999996 -0.03 rpy=0.0 -0.0 0.0
- added joint z_axis_mount_linear_rod_2: type fixed, parent z_axis_mount, child linear_rod_2, origin xyz=-0.055999999999999994 -0.06849999999999999 -0.03 rpy=0.0 -0.0 0.0
- added joint z_axis_mount_linear_rod_3: type fixed, parent z_axis_mount, child linear_rod_3, origin xyz=0.003999999999999999 -0.06849999999999999 -0.03 rpy=0.0 -0.0 0.0
- added joint z_axis_mount_linear_rod_4: type fixed, parent z_axis_mount, child linear_rod_4, origin xyz=0.003999999999999999 0.013499999999999996 -0.03 rpy=0.0 -0.0 0.0

Commit message: Removed joint 3 and 4 limits

File: SCARA.urdf (robot description, URDF)
Before this commit: robot URDF, 25 links, 24 joints
Joints:
- joint ee_51105_bearing_ee_mount: limit lower=0.0 upper=5.585054 effort=1000 velocity=1000000 -> lower=-3.141593 upper=3.141593 effort=1000 velocity=1000000
- joint l3_51105_bearing_l3_top: limit lower=-1.22173 upper=4.712389 effort=1000 velocity=1000000 -> lower=-3.141593 upper=3.141593 effort=1000 velocity=1000000

Commit message: Modified joint 3 limits

File: SCARA.urdf (robot description, URDF)
Before this commit: robot URDF, 25 links, 24 joints
Joints:
- joint l3_51105_bearing_l3_top: limit lower=-3.141593 upper=3.141593 effort=1000 velocity=1000000 -> lower=-6.28318 upper=0 effort=1000 velocity=1000000

Commit message: Added gripper

File: SCARA.urdf (robot description, URDF)
Before this commit: robot URDF, 25 links, 24 joints
Links:
- added link gripper_adapter, mass 0.259073281997157; collision mesh filename=CAD/gripper_adapter.stl scale=0.001 0.001 0.001; visual mesh filename=CAD/gripper_adapter.stl scale=0.001 0.001 0.001
- added link gripper_mount, mass 0.12491021556465158; collision mesh filename=CAD/gripper_mount.stl scale=0.001 0.001 0.001; visual mesh filename=CAD/gripper_mount.stl scale=0.001 0.001 0.001
- added link gripper_rack_left, mass 0.09055057737962392; collision mesh filename=CAD/gripper_rack.stl scale=0.001 0.001 0.001; visual mesh filename=CAD/gripper_rack.stl scale=0.001 0.001 0.001
- added link gripper_rack_right, mass 0.09055057737962392; collision mesh filename=CAD/gripper_rack.stl scale=0.001 0.001 0.001; visual mesh filename=CAD/gripper_rack.stl scale=0.001 0.001 0.001
Joints:
- added joint ee_mount_gripper_adapter: type fixed, parent ee_mount, child gripper_adapter, origin xyz=0.016 0.0 0.006000000000000005 rpy=3.141592653589793 6.162975822039155e-33 1.2228926112441607e-33
- added joint gripper_adapter_gripper_mount: type fixed, parent gripper_adapter, child gripper_mount, origin xyz=-0.04050000000000001 -0.005999999999999997 -0.014999999999999996 rpy=9.888225988704661e-33 1.0364333334546883e-47 -1.3489594288050942e-48
- added joint gripper_mount_gripper_rack_left: type fixed, parent gripper_mount, child gripper_rack_left, origin xyz=-0.0019999999999999974 -0.012800000000000011 0.013000000000000003 rpy=6.703233356227362e-16 -1.5707963267948966 0
- added joint gripper_mount_gripper_rack_right: type fixed, parent gripper_mount, child gripper_rack_right, origin xyz=0.051000000000000004 -0.012800000000000011 -0.021 rpy=-3.141592653589793 -1.5707963267948966 0
- joint ee_51105_bearing_ee_mount: limit lower=-3.141593 upper=3.141593 effort=1000 velocity=1000000 -> lower=0 upper=3.141593 effort=1000 velocity=1000000
